Commit message: buliding map an models

File: description/racecar.urdf.xacro (robot description, xacro)
@@ -1,53 +1,57 @@
 <?xml version="1.0"?>
-<robot name="racecar" xmlns:xacro="http://www.ros.org/wiki/xacro">
-  <!-- <xacro:macro name="diffbot" params="prefix"> -->
-  <!-- Constants for robot dimensions -->
-  <xacro:property name="prefix" value="racecar_"/>
-  <xacro:property name="PI" value="3.1415926535897931"/>
-  <xacro:property name="base_mass" value="0.3" /> <!-- arbitrary value for base mass -->
-  <xacro:property name="base_width" value="0.1" />
-  <xacro:property name="base_length" value="0.1" />
-  <xacro:property name="base_height" value="0.05" />
-  <xacro:property name="wheel_mass" value="0.3" /> <!-- arbitrary value for wheel mass -->
-  <xacro:property name="wheel_len" value="0.020" />
-  <xacro:property name="wheel_radius" value="0.015" />
-  <xacro:property name="caster_wheel_mass" value="0.1" /> <!-- arbitrary value for caster wheel mass -->
-  <xacro:property name="caster_wheel_radius" value="0.015" />
-  <xacro:property name="z_offset" value="-${base_height/2}" /> <!-- Space btw top of beam and the each joint -->
-  <!-- Base Link -->
-  <link name="${prefix}base_link">
-    <collision>
-      <origin xyz="0 0 0" rpy="0 0 0"/>
-      <geometry>
-        <box size="${base_width} ${base_length} ${base_height}"/>
-      </geometry>
-    </collision>
-    <visual>
-      <origin xyz="0 0 0" rpy="0 0 0"/>
-      <geometry>
-        <box size="${base_width} ${base_length} ${base_height}"/>
-      </geometry>
-      <material name="orange"/>
-    </visual>
-    <inertial>
-      <origin xyz="0 0 0" rpy="0 0 0"/>
-      <mass value="${base_mass}"/>
-      <inertia
-        ixx="${base_mass / 12.0 * (base_length*base_length + base_height*base_height)}" ixy="0.0" ixz="0.0"
-        iyy="${base_mass / 12.0 * (base_height*base_height + base_width*base_width)}" iyz="0.0"
-        izz="${base_mass / 12.0 * (base_width*base_width + base_length*base_length)}"/>
+<robot xmlns:xacro="http://www.ros.org/wiki/xacro">
+  <xacro:macro name="racecar" params="prefix">
+   <!-- Constants for robot dimensions -->
+    <xacro:property name="PI" value="3.1415926535897931"/>
+    <xacro:property name="base_mass" value="0.3" /> <!-- arbitrary value for base mass -->
+    <xacro:property name="base_width" value="0.1" />
+    <xacro:property name="base_length" value="0.1" />
+    <xacro:property name="base_height" value="0.05" />
+    <xacro:property name="wheel_mass" value="0.3" /> <!-- arbitrary value for wheel mass -->
+    <xacro:property name="wheel_len" value="0.020" />
+    <xacro:property name="wheel_radius" value="0.015" />
+    <xacro:property name="caster_wheel_mass" value="0.1" /> <!-- arbitrary value for caster wheel mass -->
+    <xacro:property name="caster_wheel_radius" value="0.015" />
+    <xacro:property name="z_offset" value="-${base_height/2}" /> <!-- Space btw top of beam and the each joint -->
+    <link name="dummy"/>
+    <joint name="dummy_joint" type="fixed">
+     <parent link="dummy"/>
+     <child link="base_link"/>
+   </joint>
+    <!-- Base Link -->
+    <link name="${prefix}base_link">
+      <collision>
+        <origin xyz="0 0 0" rpy="0 0 0"/>
+        <geometry>
+          <box size="${base_width} ${base_length} ${base_height}"/>
+        </geometry>
+      </collision>
+      <visual>
+        <origin xyz="0 0 0" rpy="0 0 0"/>
+        <geometry>
+          <box size="${base_width} ${base_length} ${base_height}"/>
+        </geometry>
+        <material name="orange"/>
+      </visual>
+      <inertial>
+        <origin xyz="0 0 0" rpy="0 0 0"/>
+        <mass value="${base_mass}"/>
+        <inertia
+          ixx="${base_mass / 12.0 * (base_length*base_length + base_height*base_height)}" ixy="0.0" ixz="0.0"
+          iyy="${base_mass / 12.0 * (base_height*base_height + base_width*base_width)}" iyz="0.0"
+          izz="${base_mass / 12.0 * (base_width*base_width + base_length*base_length)}"/>
       </inertial>
     </link>
-    <joint name="${prefix}left_wheel_joint" type="continuous">
+    <joint name="${prefix}left_wheel_joint" type="fixed">
       <parent link="${prefix}base_link"/>
       <child link="${prefix}left_wheel"/>
       <origin xyz="0 -${base_width/2} ${z_offset}" rpy="0 0 0"/>
-      <axis xyz="0 1 0"/>
-      <dynamics damping="0.2"/>
+      <!-- <axis xyz="0 1 0"/> -->
+      <!-- <dynamics damping="0.2"/> -->
     </joint>
-    <!-- left wheel Link -->
+      <!-- left wheel Link -->
     <link name="${prefix}left_wheel">
       <collision>
-        <origin xyz="0 0 0" rpy="${PI/2} 0 0"/>
+        <origin xyz="0 -${base_width/2} ${z_offset}" rpy="${PI/2} 0 0"/>
         <geometry>
           <cylinder length="${wheel_len}" radius="${wheel_radius}"/>
@@ -55,5 +59,5 @@
       </collision>
       <visual>
-        <origin xyz="0 0 0" rpy="${PI/2} 0 0"/>
+        <origin xyz="0 -${base_width/2} ${z_offset}" rpy="${PI/2} 0 0"/>
         <geometry>
           <cylinder length="${wheel_len}" radius="${wheel_radius}"/>
@@ -62,12 +66,12 @@
       </visual>
       <inertial>
-        <origin xyz="0 0 0" rpy="${PI/2} 0 0"/>
+        <origin xyz="0 -${base_width/2} ${z_offset}" rpy="${PI/2} 0 0"/>
         <mass value="${wheel_mass}"/>
         <inertia
-          ixx="${(wheel_mass / 12.0) * (3*wheel_radius*wheel_radius + (wheel_len*wheel_len))}" ixy="0.0" ixz="0.0"
-          iyy="${(wheel_mass / 12.0) * (wheel_radius*wheel_radius + wheel_len*wheel_len)}" iyz="0.0"
-          izz="${wheel_mass * (wheel_radius*wheel_radius)/2}"/>
-        </inertial>
-      </link>
+          ixx="${wheel_mass / 12.0 * (3*wheel_radius + wheel_len*wheel_len)}" ixy="0.0" ixz="0.0"
+          iyy="${wheel_mass / 12.0 * wheel_radius*wheel_radius}" iyz="0.0"
+          izz="${wheel_mass / 12.0 * wheel_radius*wheel_radius}"/>
+      </inertial>
+    </link>
     <joint name="${prefix}right_wheel_joint" type="continuous">
       <parent link="${prefix}base_link"/>
@@ -77,5 +81,5 @@
       <dynamics damping="0.2"/>
     </joint>
-    <!-- right wheel Link -->
+      <!-- right wheel Link -->
     <link name="${prefix}right_wheel">
       <collision>
@@ -96,9 +100,9 @@
         <mass value="${wheel_mass}"/>
         <inertia
-          ixx="${(wheel_mass / 12.0) * (3*wheel_radius*wheel_radius + (wheel_len*wheel_len))}" ixy="0.0" ixz="0.0"
-          iyy="${(wheel_mass / 12.0) * (wheel_radius*wheel_radius + wheel_len*wheel_len)}" iyz="0.0"
-          izz="${wheel_mass * (wheel_radius*wheel_radius)/2}"/>
-        </inertial>
-      </link>
+          ixx="${wheel_mass / 12.0 * (3*wheel_radius + wheel_len*wheel_len)}" ixy="0.0" ixz="0.0"
+          iyy="${wheel_mass / 12.0 * wheel_radius*wheel_radius}" iyz="0.0"
+          izz="${wheel_mass / 12.0 * wheel_radius*wheel_radius}"/>
+      </inertial>
+    </link>
     <joint name="${prefix}caster_frontal_wheel_joint" type="fixed">
       <parent link="${prefix}base_link"/>
@@ -106,5 +110,4 @@
       <origin xyz="${base_width/2 - caster_wheel_radius} 0 ${z_offset}" rpy="0 0 0"/>
     </joint>
-    <!-- caster frontal wheel Link -->
     <link name="${prefix}caster_frontal_wheel">
       <collision>
@@ -135,5 +138,4 @@
       <origin xyz="${-base_width/2 + caster_wheel_radius} 0 ${z_offset}" rpy="0 0 0"/>
     </joint>
-    <!-- caster rear wheel Link -->
     <link name="${prefix}caster_rear_wheel">
       <collision>
@@ -159,4 +161,4 @@
       </inertial>
     </link>
-  <!-- </xacro:macro> -->
+  </xacro:macro>
 </robot>
